Commit message: updated rviz visualization

File: visualization/abz.urdf.xacro (robot description, xacro)
@@ -2,10 +2,12 @@
 <!-- Kinematic model, simplified visual, no collisions -->
 <robot name="lab" xmlns:xacro="http://www.ros.org/wiki/xacro">
-<xacro:include filename="$(find atlas_config_abz)/visualization/materials.xacro" />
+<xacro:include filename="$(find atlas_config_celidon)/visualization/materials.xacro" />
   <link name="base_link">
    <visual>
       <geometry>
-        <mesh scale=".001 .001 .001" filename="file://$(find atlas_config_abz)/visualization/abz.stl"/>
+        <mesh scale=".001 .001 .001" filename="file://$(find atlas_config_celidon)/visualization/abz.stl"/>
       </geometry>
+      <origin xyz="-10 -5 -4"/>
+      <material name="Grey"/>
    </visual>
   </link>

File: visualization/materials.xacro (robot description, xacro)
@@ -1,4 +1,4 @@
 <?xml version="1.0"?>
-<material name="Orange">
-	<color rgba="${255/255} ${108/255} ${10/255} 1.0"/>
+<material name="Grey">
+	<color rgba="${250/255} ${250/255} ${250/255} 1.0"/>
 </material>
